Commit message: play with exporter

File: code/src/u1/urdf/robot.urdf (robot description, URDF)
Before this commit: robot robot, 2 links, 1 joints
Links:
- removed link Bottom
- removed link base_link
- added link box1; visual mesh filename=package://u1/meshes/box1.stl scale=0.001 0.001 0.001
- added link box2; visual mesh filename=package://u1/meshes/box2.stl scale=0.001 0.001 0.001
Joints:
- removed joint gripper_extension
